File: OLED-Clock-6-nl.brd (EAGLE design)
At the start: 27.3 x 26.9 mm, 30 parts, among them IC1 ATMEGA328P, IC2 DS3231MZ, T1 FDC6327C

Commit message: Add files via upload
Parts:
- removed DSP1: DISPLAY-OLED-128X64-I2C, diy-modules:DISPLAY-OLED-128X64-I2C
- removed JP1: AVR-ISP-6, avr-7:AVR-ISP-6
- removed S1, S2: DTSM-3, switch-tact:DTSM-3
Connections:
- net A4_SDA: no longer DSP1.4
- net A5_SCL: no longer DSP1.3
- net GND: no longer DSP1.1, JP1.6, S1.2, S2.2
- net MISO: no longer JP1.1
- net MOSI: no longer JP1.4
- net N$1: no longer S1.1
- net N$6: no longer S2.1
- net RST: no longer JP1.5
- net SCK: no longer JP1.3
- net VCC: no longer DSP1.2, JP1.2
Routing:
- net GND: track 122.2 -> 111.9 mm
- net N$6: track 17.7 -> 15.9 mm
- net N$1: track 5.38 -> 4.49 mm
- net A5_SCL: track 12.5 -> 11.6 mm
- net VCC: track 53.2 -> 52.5 mm
Other:
- outline, holes or cut-outs redrawn
- board text added: "1. Batt. (CR2430) bottom 2. ATmega-Board mean 3. OLED-Display top"
- board text removed: "(from above)"
- board text removed: "1. Batt. (CR2430) bottom 2. ATmega-Board top 3. OLED-Display top"
- board text removed: "Batt. +/-Conn. (reversed)"
- board text removed: "LED: 1,4x3,0mm"
- board text removed: "MOSI"
- board text removed: "OLED + LED1 (on top)"
- board text removed: "Socket-header"
- board text removed: "Socket-header:"
- board text removed: "Vias:"
- board text removed: "Wire:"
- board text removed: "o4mm"
- board text removed: "o5mm"
