File: OLED-Clock-6-nl.sch (EAGLE design)
At the start: 26 parts, among them IC1 ATMEGA328P, IC2 DS3231MZ, T1 FDC6327C

Commit message: Add files via upload
Other:
- note added: "Dual N+P-Mosfet"
Changed lines of the file:
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@@
 <setting verticaltext="up"/>
 </settings>
-<grid distance="0.1" unitdist="inch" unit="inch" style="lines" multiple="1" display="no" altdistance="0.01" altunitdist="inch" altunit="inch"/>
+<grid distance="0.025" unitdist="inch" unit="inch" style="dots" multiple="1" display="yes" altdistance="0.01" altunitdist="inch" altunit="inch"/>
 <layers>
 <layer number="1" name="Top" color="4" fill="1" visible="no" active="no"/>
@@
 <wire x1="147.32" y1="37.465" x2="147.32" y2="35.56" width="0.1524" layer="94" style="shortdash"/>
 <text x="143.51" y="39.6875" size="1.778" layer="95">S2</text>
+<text x="196.85" y="167.005" size="1.778" layer="97">Dual N+P-Mosfet</text>
 </plain>
 <instances>
